Commit message: updating urdf for sim

File: vector_common/vector_description/urdf/sensors/sick_tim.urdf.xacro (robot description, xacro)
@@ -36,5 +36,5 @@
             <collision>
                 <geometry>
-                    <box size="0.1 0.1 0.1"/>
+                    <box size="0.05 0.05 0.05"/>
                 </geometry>
             </collision>
@@ -55,7 +55,7 @@
                     </scan>
                     <range>
-                        <min>0.05</min>
+                        <min>0.06</min>
                         <max>10.0</max>
-                        <resolution>0.01</resolution>
+                        <resolution>0.001</resolution>
                     </range>
                     <noise>
