Commit message: updating hokuyo uam model for sim

File: vector_common/vector_description/urdf/sensors/hokuyo_uam_05lp.urdf.xacro (robot description, xacro)
@@ -36,5 +36,5 @@
             <collision>
                 <geometry>
-                    <box size="0.1 0.1 0.1"/>
+                    <box size="0.05 0.05 0.05"/>
                 </geometry>
             </collision>
@@ -55,5 +55,5 @@
                     </scan>
                     <range>
-                        <min>0.05</min>
+                        <min>0.06</min>
                         <max>20.0</max>
                         <resolution>0.01</resolution>
