Commit message: making laser positions and ranges fixed for each type

File: vector_common/vector_description/urdf/accessories.urdf.xacro (robot description, xacro)
@@ -48,8 +48,8 @@
         <xacro:unless value="$(optenv VECTOR_HAS_SAFETY_LASERS false)">
             <xacro:sick_tim laser_prefix="front" parent="base_chassis_link">
-                <origin xyz="0.3075 0 0.1439106" rpy="3.14159 0 0" />
+                <origin xyz="0.2525 0.1918 0.13791" rpy="${M_PI} 0 ${M_PI/4}" />
             </xacro:sick_tim>
             <xacro:sick_tim laser_prefix="rear" parent="base_chassis_link">
-                <origin xyz="-0.3075 0 0.1439106" rpy="3.14159 0 3.14159" />
+                <origin xyz="-0.2525 -0.1918 0.13791" rpy="${M_PI} 0 ${5*M_PI/4}" />
             </xacro:sick_tim>
         </xacro:unless>

File: vector_common/vector_description/urdf/sensors/hokuyo_uam_05lp.urdf.xacro (robot description, xacro)
@@ -50,10 +50,10 @@
                         <samples>720</samples>
                         <resolution>1</resolution>
-                        <min_angle>-2.36</min_angle>
-                        <max_angle>2.36</max_angle>
+                        <min_angle>-2.356</min_angle>
+                        <max_angle>2.356</max_angle>
                         </horizontal>
                     </scan>
                     <range>
-                        <min>0.1</min>
+                        <min>0.05</min>
                         <max>20.0</max>
                         <resolution>0.01</resolution>

File: vector_common/vector_description/urdf/sensors/sick_tim.urdf.xacro (robot description, xacro)
@@ -50,11 +50,11 @@
                         <samples>720</samples>
                         <resolution>1</resolution>
-                        <min_angle>-1.5708</min_angle>
-                        <max_angle>1.5708</max_angle>
+                        <min_angle>-2.35619449</min_angle>
+                        <max_angle>2.35619449</max_angle>
                         </horizontal>
                     </scan>
                     <range>
-                        <min>0.1</min>
-                        <max>25.0</max>
+                        <min>0.05</min>
+                        <max>10.0</max>
                         <resolution>0.01</resolution>
                     </range>

Commit message: adding description for si_dev machine

File: vector_common/vector_description/urdf/accessories.urdf.xacro (robot description, xacro)
@@ -46,20 +46,30 @@
             </plugin>
         </gazebo>
-        <xacro:unless value="$(optenv VECTOR_HAS_SAFETY_LASERS false)">
+        <xacro:if value="$(optenv SI_DEV_VECTOR false)">
             <xacro:sick_tim laser_prefix="front" parent="base_chassis_link">
-                <origin xyz="0.2525 0.1918 0.13791" rpy="${M_PI} 0 ${M_PI/4}" />
+                <origin xyz="0.306500 0 0.142068" rpy="${M_PI} 0 0" />
             </xacro:sick_tim>
             <xacro:sick_tim laser_prefix="rear" parent="base_chassis_link">
-                <origin xyz="-0.2525 -0.1918 0.13791" rpy="${M_PI} 0 ${5*M_PI/4}" />
+                <origin xyz="-0.306500 0 0.142068" rpy="${M_PI} 0 ${M_PI}" />
             </xacro:sick_tim>
+        </xacro:if>
+        <xacro:unless value="$(optenv SI_DEV_VECTOR false)">
+            <xacro:unless value="$(optenv VECTOR_HAS_SAFETY_LASERS false)">
+                <xacro:sick_tim laser_prefix="front" parent="base_chassis_link">
+                    <origin xyz="0.2525 0.1918 0.13791" rpy="${M_PI} 0 ${M_PI/4}" />
+                </xacro:sick_tim>
+                <xacro:sick_tim laser_prefix="rear" parent="base_chassis_link">
+                    <origin xyz="-0.2525 -0.1918 0.13791" rpy="${M_PI} 0 ${5*M_PI/4}" />
+                </xacro:sick_tim>
+            </xacro:unless>
+            <xacro:if value="$(optenv VECTOR_HAS_SAFETY_LASERS false)">
+                <xacro:hokuyo_uam_05lp laser_prefix="front" parent="base_chassis_link">
+                    <origin xyz="0.252995 0.192212 0.137128" rpy="${M_PI} 0 ${M_PI/4}"/>
+                </xacro:hokuyo_uam_05lp>
+                <xacro:hokuyo_uam_05lp laser_prefix="rear" parent="base_chassis_link">
+                    <origin xyz="-0.252995 -0.192212 0.137128" rpy="${M_PI} 0 ${5*M_PI/4}" />
+                </xacro:hokuyo_uam_05lp>
+            </xacro:if>
         </xacro:unless>
-        <xacro:if value="$(optenv VECTOR_HAS_SAFETY_LASERS false)">
-            <xacro:hokuyo_uam_05lp laser_prefix="front" parent="base_chassis_link">
-                <origin xyz="0.252995 0.192212 0.137128" rpy="${M_PI} 0 ${M_PI/4}"/>
-            </xacro:hokuyo_uam_05lp>
-            <xacro:hokuyo_uam_05lp laser_prefix="rear" parent="base_chassis_link">
-                <origin xyz="-0.252995 -0.192212 0.137128" rpy="${M_PI} 0 ${5*M_PI/4}" />
-            </xacro:hokuyo_uam_05lp>
-        </xacro:if>
     </xacro:macro>
 </robot>

File: vector_common/vector_description/urdf/vector_components/vector_base.urdf.xacro (robot description, xacro)
@@ -41,13 +41,27 @@
 	    </inertial>
             <collision>
-				<geometry>
-					<mesh filename="package://vector_description/meshes/vector_components/collision/vector_base_collision.stl" />
-				</geometry>
+                <xacro:if value="$(optenv SI_DEV_VECTOR false)">
+				    <geometry>
+					    <mesh filename="package://vector_description/meshes/vector_components/collision/vector_bw_base_collision.stl" />
+				    </geometry>
+				</xacro:if>
+                <xacro:unless value="$(optenv SI_DEV_VECTOR false)">
+				    <geometry>
+					    <mesh filename="package://vector_description/meshes/vector_components/collision/vector_base_collision.stl" />
+				    </geometry>
+				</xacro:unless>
 			</collision>
 			<visual>
 				<origin xyz="0 0 0" rpy="0 0 0" />
-				<geometry>
-					<mesh filename="package://vector_description/meshes/vector_components/visual/vector_base.dae" />
-				</geometry>
+                <xacro:if value="$(optenv SI_DEV_VECTOR false)">
+				    <geometry>
+					    <mesh filename="package://vector_description/meshes/vector_components/visual/vector_bw_base.dae" />
+				    </geometry>
+				</xacro:if>
+                <xacro:unless value="$(optenv SI_DEV_VECTOR false)">
+				    <geometry>
+					    <mesh filename="package://vector_description/meshes/vector_components/visual/vector_base.dae" />
+				    </geometry>
+				</xacro:unless>
 			</visual>
 		</link>
@@ -73,13 +87,27 @@
 			</inertial>
             <collision>
-				<geometry>
-					<mesh filename="package://vector_description/meshes/vector_components/collision/std_payload_plate_collision.stl" />
-				</geometry>
+                <xacro:if value="$(optenv SI_DEV_VECTOR false)">
+				    <geometry>
+					    <mesh filename="package://vector_description/meshes/vector_components/collision/dev_payload_plate_collision.stl" />
+				    </geometry>
+				</xacro:if>
+                <xacro:unless value="$(optenv SI_DEV_VECTOR false)">
+				    <geometry>
+					    <mesh filename="package://vector_description/meshes/vector_components/collision/std_payload_plate_collision.stl" />
+				    </geometry>
+				</xacro:unless>
 			</collision>
 			<visual>
 				<origin xyz="0 0 0" rpy="0 0 0" />
-				<geometry>
-					<mesh filename="package://vector_description/meshes/vector_components/visual/std_payload_plate.dae" />
-				</geometry>
+                <xacro:if value="$(optenv SI_DEV_VECTOR false)">
+				    <geometry>
+					    <mesh filename="package://vector_description/meshes/vector_components/visual/dev_payload_plate.dae" />
+				    </geometry>
+				</xacro:if>
+                <xacro:unless value="$(optenv SI_DEV_VECTOR false)">
+				    <geometry>
+					    <mesh filename="package://vector_description/meshes/vector_components/visual/std_payload_plate.dae" />
+				    </geometry>
+				</xacro:unless>
 			</visual>
 		</link>

Commit message: adding VLP16 to urdf

File: vector_common/vector_description/urdf/accessories.urdf.xacro (robot description, xacro)
@@ -24,4 +24,6 @@
     <xacro:include filename="$(find vector_description)/urdf/sensors/sick_tim.urdf.xacro"/>
     <xacro:include filename="$(find vector_description)/urdf/sensors/hokuyo_uam_05lp.urdf.xacro"/>
+    <xacro:include filename="$(find vector_description)/urdf/sensors/velodyne_vlp16.urdf.xacro"/>
+    <xacro:include filename="$(find vector_description)/urdf/vector_components/vector_vlp16_mount.urdf.xacro"/>
     <xacro:property name="M_PI" value="3.14159"/>
     <xacro:macro name="vector_accessories">
@@ -72,4 +74,10 @@
             </xacro:if>
         </xacro:unless>
+        <xacro:if value="$(optenv VECTOR_HAS_VLP16 false)">
+            <xacro:vector_vlp16_mount/>
+            <xacro:velodyne_vlp16 parent="base_chassis_link">
+                <origin xyz="0 0 0.315507" rpy="0 0 0" />
+            </xacro:velodyne_vlp16>
+        </xacro:if>
     </xacro:macro>
 </robot>

File: vector_common/vector_description/urdf/vector_components/vector_base.urdf.xacro (robot description, xacro)
@@ -112,5 +112,5 @@
 			</visual>
 		</link>
-        <gazebo reference="base_chassis_link">
+        <gazebo reference="payload_plate_link">
 			<mu1 value="0.3"/>
 			<mu2 value="0.3"/>

Commit message: Added modified Velodyne Laserscan. Added Webcam config.

File: vector_common/vector_description/urdf/accessories.urdf.xacro (robot description, xacro)
@@ -83,5 +83,7 @@
         </xacro:if>
         <xacro:if value="$(optenv VECTOR_HAS_WEBCAM false)">
-            <xacro:webcam parent="base_chassis_link"/>
+            <xacro:webcam parent="base_chassis_link">
+                <origin xyz="0.27 0 0.09" rpy="0 0 0"/>
+            </xacro:webcam>
         </xacro:if>
         <xacro:if value="$(optenv VECTOR_HAS_REALSENSE false)">

File: vector_common/vector_description/urdf/sensors/webcam.urdf.xacro (robot description, xacro)
@@ -2,8 +2,7 @@
 <robot xmlns:xacro="http://ros.org/wiki/xacro" name="webcam">
  <xacro:property name="camera_link" value="0.05" /> <!-- Size of square 'camera' box -->
- <xacro:macro name="webcam" params="parent">
+ <xacro:macro name="webcam" params="parent *origin">
   <joint name="camera_joint" type="fixed">
-    <axis xyz="0 1 0" />
-    <origin xyz="0.27 0 0.09" rpy="0 0 0"/>
+    <xacro:insert_block name="origin" />
     <parent link="${parent}"/>
     <child link="camera_link"/>
@@ -29,4 +28,13 @@
       <inertia ixx="1e-6" ixy="0" ixz="0" iyy="1e-6" iyz="0" izz="1e-6" />
     </inertial>
+  </link>
+  <joint name="camera_optical_joint" type="fixed">
+    <origin xyz="0 0 0" rpy="${-pi/2} 0 ${-pi/2}"/>
+    <parent link="camera_link"/>
+    <child link="camera_link_optical"/>
+  </joint>
+  <link name="camera_link_optical">
+  <!-- This link exists for the real world cameras. OpenCV uses a different axis
+  convention than the virtual camera in gazebo, hence the "optical" link -->
   </link>
 <!-- camera -->
