Commit message: adding wheel type to vector config
possible values are HD and standard

File: vector_common/vector_description/urdf/vector_components/vector_base.urdf.xacro (robot description, xacro)
@@ -24,4 +24,5 @@
     <!-- Wheel Mounting Positions and Properties-->
     <xacro:property name="wheel_radius" value="0.0762" />
+    <xacro:property name="wheel_type" value="$(optenv VECTOR_WHEEL_TYPE standard)"/>
 	<xacro:macro name="vector_base">
         <!-- Base link is the center of the robot's chassis between the motors projected on the ground -->
@@ -41,27 +42,27 @@
 	    </inertial>
             <collision>
-                <xacro:if value="$(optenv SI_DEV_VECTOR false)">
+                <xacro:if value="${wheel_type == 'HD'}">
 				    <geometry>
 					    <mesh filename="package://vector_description/meshes/vector_components/collision/vector_bw_base_collision.stl" />
 				    </geometry>
 				</xacro:if>
-                <xacro:unless value="$(optenv SI_DEV_VECTOR false)">
+                <xacro:if value="${wheel_type == 'standard'}">
 				    <geometry>
 					    <mesh filename="package://vector_description/meshes/vector_components/collision/vector_base_collision.stl" />
 				    </geometry>
-				</xacro:unless>
+				</xacro:if>
 			</collision>
 			<visual>
 				<origin xyz="0 0 0" rpy="0 0 0" />
-                <xacro:if value="$(optenv SI_DEV_VECTOR false)">
+                <xacro:if value="${wheel_type == 'HD'}">
 				    <geometry>
 					    <mesh filename="package://vector_description/meshes/vector_components/visual/vector_bw_base.dae" />
 				    </geometry>
 				</xacro:if>
-                <xacro:unless value="$(optenv SI_DEV_VECTOR false)">
+                <xacro:if value="${wheel_type == 'standard'}">
 				    <geometry>
 					    <mesh filename="package://vector_description/meshes/vector_components/visual/vector_base.dae" />
 				    </geometry>
-				</xacro:unless>
+				</xacro:if>
 			</visual>
 		</link>
